Commit message: feat(gazebo): T027-T029 Add simulated LiDAR, Camera, and IMU to humanoid URDF

File: code/module1/humanoid_description/urdf/humanoid.urdf (robot description, URDF)
Before this commit: robot humanoid, 16 links, 15 joints
Links:
- added link imu_link, mass 0.01; collision box size=0.02 0.02 0.01; visual box size=0.02 0.02 0.01
- added link lidar_link, mass 0.1; collision cylinder length=0.05 radius=0.03; visual cylinder length=0.05 radius=0.03
- added link realsense_d435_link, mass 0.05; collision box size=0.01 0.09 0.025; visual box size=0.01 0.09 0.025
Joints:
- added joint head_to_imu: type fixed, parent head, child imu_link, origin xyz=-0.03 0 0.08 rpy=0 0 0
- added joint head_to_lidar: type fixed, parent head, child lidar_link, origin xyz=0 0 0.08 rpy=0 0 0
- added joint head_to_realsense: type fixed, parent head, child realsense_d435_link, origin xyz=0 0.04 0.08 rpy=0 0 0
